Commit message: launch/raspicat_navigation.launch start_motor.launch add
param/costmap_common_params_burger.yaml
robot range param change

param/dwa_local_planner_params_burger.yaml
param change

param/global_costmap_params.yaml
robot_base_frame & transform_tolerance fix

param/local_costmap_params.yaml
window & transform_tolerance fix

rviz/raspicat_navigation.rviz
2D->3Dview

urdf/raspicat.urdf.xacro
base_footprint remove

File: urdf/raspicat.urdf.xacro (robot description, xacro)
@@ -16,17 +16,4 @@
     </inertial>
   </link>
-  <link name="imu_link">
-    <visual>
-      <origin xyz="0 0 0" />
-      <geometry>
-        <box size="0.06 0.04 0.02" />
-      </geometry>
-    </visual>
-  </link>
-  <joint name="imu_joint" type="fixed">
-    <parent link="base_link"/>
-    <child link="imu_link"/>
-    <origin xyz="0 0 0" rpy="0 0 0"/>
-  </joint>
   <joint name="scan_joint" type="fixed">
     <parent link="base_link"/>

Commit message: change urdf

File: urdf/raspicat.urdf.xacro (robot description, xacro)
@@ -1,27 +1,12 @@
 <?xml version="1.0" ?>
-<robot name="turtlebot3_burger" xmlns:xacro="http://ros.org/wiki/xacro">
-  <link name="base_link">
-    <collision>
-      <origin xyz="-0.032 0 0.070" rpy="0 0 0"/>
-      <geometry>
-        <box size="0.140 0.140 0.143"/>
-      </geometry>
-    </collision>
-    <inertial>
-      <origin xyz="0 0 0" rpy="0 0 0"/>
-      <mass value="8.2573504e-01"/>
-      <inertia ixx="2.2124416e-03" ixy="-1.2294101e-05" ixz="3.4938785e-05"
-               iyy="2.1193702e-03" iyz="-5.0120904e-06"
-               izz="2.0064271e-03" />
-    </inertial>
-  </link>
-  <link name="imu_link">
-    <visual>
-      <origin xyz="0 0 0" />
-      <geometry>
-        <box size="0.06 0.04 0.02" />
-      </geometry>
-    </visual>
-  </link>
+<robot name="raspicat" xmlns:xacro="http://ros.org/wiki/xacro">
+  <link name="base_footprint"/>
+  <joint name="base_joint" type="fixed">
+    <parent link="base_footprint"/>
+    <child link="base_link"/>
+    <origin xyz="0.0 0.0 0.05" rpy="0 0 0"/>
+  </joint>
+  <link name="base_link"/>
+  <link name="imu_link"/>
   <joint name="imu_joint" type="fixed">
     <parent link="base_link"/>
@@ -29,23 +14,9 @@
     <origin xyz="0 0 0" rpy="0 0 0"/>
   </joint>
-  <joint name="scan_joint" type="fixed">
+  <joint name="urg_joint" type="fixed">
     <parent link="base_link"/>
     <child link="urg_lrf_link"/>
-    <origin xyz="-0.032 0 0.172" rpy="0 0 0"/>
+    <origin xyz="0.144 0.0 0.04" rpy="0 0 0"/>
   </joint>
-  <link name="urg_lrf_link">
-    <collision>
-      <origin xyz="0.015 0 -0.0065" rpy="0 0 0"/>
-      <geometry>
-        <cylinder length="0.0315" radius="0.055"/>
-      </geometry>
-    </collision>
-    <inertial>
-      <mass value="0.114" />
-      <origin xyz="0 0 0" />
-      <inertia ixx="0.001" ixy="0.0" ixz="0.0"
-               iyy="0.001" iyz="0.0"
-               izz="0.001" />
-    </inertial>
-  </link>
+  <link name="urg_lrf_link"/>
 </robot>

Commit message: changed base_joint

File: urdf/raspicat.urdf.xacro (robot description, xacro)
@@ -5,5 +5,5 @@
     <parent link="base_footprint"/>
     <child link="base_link"/>
-    <origin xyz="0.0 0.0 0.05" rpy="0 0 0"/>
+    <origin xyz="0.0 0.0 0.0762" rpy="0 0 0"/>
   </joint>
   <link name="base_link"/>

Commit message: imu_joint 0->x 0->z

File: urdf/raspicat.urdf.xacro (robot description, xacro)
@@ -12,5 +12,5 @@
     <parent link="base_link"/>
     <child link="imu_link"/>
-    <origin xyz="0 0 0" rpy="0 0 0"/>
+    <origin xyz="0.008 0 13.4" rpy="0 0 0"/>
   </joint>
   <joint name="urg_joint" type="fixed">

Commit message: imu_linkの修正

File: urdf/raspicat.urdf.xacro (robot description, xacro)
@@ -12,5 +12,5 @@
     <parent link="base_link"/>
     <child link="imu_link"/>
-    <origin xyz="0.008 0 13.4" rpy="0 0 0"/>
+    <origin xyz="0 0 0.16" rpy="0 0 0"/>
   </joint>
   <joint name="urg_joint" type="fixed">
